File: V2/L2_board.kicad_pcb (KiCad board)
At the start: 4 copper layers, 101.6 x 26.9 mm, 64 parts, among them J1 SPI_Interface_Male, J2 USB_B_Micro, J3 RRC3, J4 THD2528-11SD-GF, J6 Conn_Coaxial, J7 FTDI_Female, J8 I2C_Interface_Male, J9 2-3S_LiPo_LARGE_HOLE_XT-30, Q1 Si2301CDS, Q2 MMBT2222, Q3 MMBT2222, Q4 MMBT2222, SW1 BOOT, U1 ESP32-WROOM-32, U2 AMS1117-3.3, U3 MS5611, U4 CP2102N-A01-GQFN28, U5 L80-M39, U6 MPU-6050, U7 RFM95W-915S2

Commit message: Updated costing sheet:
Other:
- net class Default removed
